File: Hardware/APPMC.sch (KiCad schematic (older format))
At the start: 117 parts, among them J1 + 30V max, J10 STLINK-V3, J101 ADC_C, J102 ADC_D, J11 Waveshare 14747, J12 I2C, J13 Micro-USB B, J14 VDD, J15 PWM, J16 ADC_B, J17 3.0V, J18 1.5V, J19 DAC_A, J2 VOut, J20 ADC_A, J21 DAC_B, J22 Jumper-2B-Open, J23 GND, J24 Jumper-2B-Open, J3 Jumper-2B-Open, J4 Jumper-2B-Open, J6 STLINK-V2, J7 VCC, J8 Conn_01x04, J9 Waveshare 18179, M4 Logo_Open_Hardware_Small, Q1 SI2343CDS-T1-GE3, Q2 ZXMP4A16GTA, Q3 ZXMP4A16GTA, Q4 BSS123, SW1 RESET, U1 INA823, U101 OPA320, U2 3.3V, U3 REF2030, U4 MAX12931, U5 STM32G0B1CEUx, U6 24CW640T-I/OT, U7 USBLC6-4SC6, U8 OPA378/387/392, U9 OPA378/387/392, Y1 32.768kHz

Commit message: docs/license info update
Parts:
- M4: footprint Symbol:KiCad-Logo2_6mm_SilkScreen -> Symbol:KiCad-Logo2_5mm_SilkScreen
Other:
- note added: "3"
- note added: "License: CC BY-NC-ND 4.0"

Commit message: MPU list errata
Other:
- note added: "alternative, pin-compatible MPUs, min 64k flash, 44-IO:\nSTM32G031C8Tx/Ux\nSTM32G041C8Tx/Ux\nSTM32G051C8Tx/Ux\nSTM32G061C8Tx/Ux\nSTM32G071C8Tx/Ux\nSTM32G071CBTx/Ux (128K)\nSTM32G081CBTx/Ux (128K)\nSTM32G0B1CBTx/Ux (128K)\nSTM32G0B1CCTx/Ux (256K)\nSTM32G0B1CETx/Ux (512k)"
- note removed: "MPU requirements: min 64kB Flash and VBAT input -> STM32G0/STM32F4 series in 48pin package"
- note removed: "alternative, pin-compatible MPUs:\nSTM32G031F8Px/G8Ux\nSTM32G041F8Px/G8Ux\nSTM32G051F8Px/G8Ux\nSTM32G061F8Px/G8Ux\nSTM32G071G8Ux/GBUx\nSTM32G081GBUx"

Commit message: values adjusted
Parts:
- R9: value 3.44k -> 3.4k
Connections:
- net labels added: 22-53Ω 21-450°C
- net labels removed: 22.65-53Ω 20-450°C (37.5 avg)
Other:
- note added: "-32.51/+37.67mV"
- note added: "0.511÷2.66V"
- note added: "1.5V"
- note added: "gain=1+(100k/Rg)=30.41"
- note removed: "+32.5/-37.7mV"
- note removed: "gain=1+(100k/Rg)=30.07"
- note removed: "~~0.5÷2.9V"
Changed lines of the file:
@@
 P 2650 7250
 F 0 "#TH1" V 2750 7200 50  0000 L CNN
-F 1 "22.65-53Ω 20-450°C (37.5 avg)" V 2500 6900 50  0000 L CNN
+F 1 "22-53Ω 21-450°C" V 2500 6900 50  0000 L CNN
 F 2 "" H 2650 7250 50  0001 C CNN
 F 3 "~" H 2650 7250 50  0001 C CNN
@@
 	1850 5550 2200 5550
 Text Notes 3700 6850 0    50   ~ 0
-gain=1+(100k/Rg)=30.07
+gain=1+(100k/Rg)=30.41
 Wire Wire Line
 	2200 6250 2450 6250
@@
 Wire Wire Line
 	1400 5550 1850 5550
-Text Notes 3700 6750 0    50   Italic 0
-+32.5/-37.7mV
 Wire Wire Line
 	2450 7250 2450 6950
@@
 	8250 4950 8300 4950
 $Comp
-L Connector:Conn_01x01_Female J20
-U 1 1 6240A578
-P 5900 6450
-F 0 "J20" H 5750 6600 50  0000 L CNN
-F 1 "ADC_A" H 5700 6400 50  0000 L CNN
-F 2 "Custom:PinHeader_1x01_P1.27mm_Vertical" H 5900 6450 50  0001 C CNN
-F 3 "~" H 5900 6450 50  0001 C CNN
-	1    5900 6450
-	1    0    0    -1
-$EndComp
-$Comp
 L Connector:Conn_01x01_Female J18
 U 1 1 61B8CE07
@@
 P 4300 6350
 F 0 "R9" V 4150 6350 50  0000 C CNN
-F 1 "3.44k" V 4400 6400 50  0000 C CNN
+F 1 "3.4k" V 4400 6400 50  0000 C CNN
 F 2 "Custom:R_0805_2012Metric_Pad1.20x1.40mm_HandSolder_Jump" H 4300 6350 50  0001 C CNN
 F 3 "~" H 4300 6350 50  0001 C CNN
@@
 $EndBitmap
 Text Notes 5350 6350 0    50   ~ 0
-~~0.5÷2.9V
+0.511÷2.66V
 Text Notes 1950 6400 0    50   ~ 0
 3.0V
@@
 Text Notes 10600 7650 0    59   ~ 12
 3
+Text Notes 3700 6750 0    50   Italic 0
+-32.51/+37.67mV
+$Comp
+L Connector:Conn_01x01_Female J20
+U 1 1 6240A578
+P 5900 6450
+F 0 "J20" H 5800 6300 50  0000 L CNN
+F 1 "ADC_A" H 5700 6400 50  0000 L CNN
+F 2 "Custom:PinHeader_1x01_P1.27mm_Vertical" H 5900 6450 50  0001 C CNN
+F 3 "~" H 5900 6450 50  0001 C CNN
+	1    5900 6450
+	1    0    0    -1
+$EndComp
+Text Notes 3650 6250 0    50   ~ 0
+1.5V
 $EndSCHEMATC

Commit message: docs update
Other:
- note added: "0.511÷2.65V"
- note removed: "0.511÷2.66V"

Commit message: docs & VS Code settings update
Connections:
- net labels added: 22-53Ω (21-450°C)
- net labels removed: 22-53Ω 21-450°C

Commit message: updates to 3.1
Connections:
- net labels removed: WKUP
- wire segments 371 -> 370

Commit message: update to 3.1
Other:
- note added: "3.1"
- note removed: "3"

Commit message: update
Parts:
- U101: value OPA320 -> OPA388
- U8, U9: value OPA378/387/392 -> OPA388
Connections:
- net labels added: 22÷53Ω (21÷450°C)
- net labels removed: 22-53Ω (21-450°C)
Other:
- note added: "R1÷R10 high grade 0.1% resistors"
- note added: "To drive light capacitive load use OPA388, NCS2005,\nOPA350EA/OPA2350EA (up to 1µF, MSOP-8 pkg)\nLM8261 (unlimited capacitive load, lower precision)"
- note added: "any low-offset (<0.1mV),\nhigh output current OpAmp\n*high CLoad drive*\nOPA388, NCS2005 (light capacitive load)\nOPA350EA (up to 1µF, MSOP-8 pkg)\nLM8261 (unlimited capacitive load use, lower precision)"
- note added: "consider driving EN from MPU"
- note added: "for WSP80 use socket: Amphenol T 3437 000"
- note added: "instead of REF2030 a) internal MPU 2.5V VREFBUF\ncan be used with divider and buffers (OpAmps),\nb) DACs can be used as Vref sources as well"
- note added: "low-offset (<0.1mV) OpAmp with low output swing headroom to negative supply (<10mV):\n- OPA387 (SOT23-5, VSSOP-8 double, TSSOP-14 quad)\n- OPA378 (SOT23-5, SC70-5, SOT23-8 double)\n- OPA391, 396 (SC70-5 only)\n- OPA320\n- OPA392 (SOT23-5, SC70-5, higher swing headroom to negative supply (~~20mV)\n"
- note added: "recommended: INA118, 317, 333, 823\noptional: INA122, 126 (two op-amp architecture\n→ limited common-mode voltage range)"
- note removed: "13992 - mono 128x128 1.5"\nsame dimensions as 14747 but 8-pin :/\n13892 - 1.8" color LCD"
- note removed: "R1-R10 high grade 0.1% resistors"
- note removed: "any low-offset (<0.1mV),\nhigh output current OpAmp"
- note removed: "for WSP80 use socket Amphenol T 3437 000"
- note removed: "https://www.waveshare.com\nSKU: 14747*"
- note removed: "https://www.waveshare.com\nSKU: 18179*"
- note removed: "instead of REF2030 internal MPU 2.5V VREFBUF\ncan be used with divider and buffers (OpAmps)"
- note removed: "low-offset (<0.1mV) OpAmp with low output swing headroom to negative supply (<10mV):\n- OPA387 (SOT23-5, VSSOP-8 double, TSSOP-14 quad)\n- OPA378 (SOT23-5, SC70-5, SOT23-8 double)\n- OPA391, 396 (SC70-5 only)\n- OPA320\n- OPA392 (SOT23-5, SC70-5, higher swing headroom to negative supply (~~20mV)"
- note removed: "recommended: INA118, 333, *823* (best option)\noptional: INA122, 126 (two op-amp architecture,\nlimited common-mode voltage range)"
