File: Hardware/APPMC.sch (KiCad schematic (older format))
At the start: 117 parts, among them J1 + 30V max, J10 STLINK-V3, J101 ADC_C, J102 ADC_D, J11 Waveshare 14747, J12 I2C, J13 Micro-USB B, J14 VDD, J15 PWM, J16 ADC_B, J17 3.0V, J18 1.5V, J19 DAC_A, J2 VOut, J20 ADC_A, J21 DAC_B, J22 Jumper-2B-Open, J23 GND, J24 Jumper-2B-Open, J3 Jumper-2B-Open, J4 Jumper-2B-Open, J6 STLINK-V2, J7 VCC, J8 Conn_01x04, J9 Waveshare 18179, M4 Logo_Open_Hardware_Small, Q1 SI2343CDS-T1-GE3, Q2 ZXMP4A16GTA, Q3 ZXMP4A16GTA, Q4 BSS123, SW1 RESET, U1 INA823, U101 OPA388, U2 3.3V, U3 REF2030, U4 MAX12931, U5 STM32G0B1CEUx, U6 24CW640T-I/OT, U7 USBLC6-4SC6, U8 OPA388, U9 OPA388, Y1 32.768kHz

Commit message: update
Other:
- note added: "any low-offset (<0.1mV),\nhigh output current OpAmp\n*high CLoad drive*\nOPA388, NCS2005 (light capacitive load)\nOPA350EA (up to 1µF, MSOP-8 pkg)\nLM8261 (unlimited capacitive load, lower precision)"
- note removed: "any low-offset (<0.1mV),\nhigh output current OpAmp\n*high CLoad drive*\nOPA388, NCS2005 (light capacitive load)\nOPA350EA (up to 1µF, MSOP-8 pkg)\nLM8261 (unlimited capacitive load use, lower precision)"

Commit message: 2022-09
Parts:
- ENC1: value Rotary_Encoder_Switch_with_MP -> PEC16-4220F-S0024
Other:
- note added: "Connector Samtec SLW-107-01-T-S"
- note added: "IR=30÷40nA@3.3V"
- note added: "To drive light capacitive load (1nF) use OPA388, NCS2005,\nOPA350EA/OP1177ARM (up to 1µF, MSOP-8 pkg)\nOPA2350EA/OP2177ARM (up to 1µF, MSOP-8 pkg, double)\nLM8261 (unlimited capacitive load, lower precision)"
- note added: "any low-offset (<0.1mV),\nhigh output current OpAmp\n*high CLoad drive*\nOPA388, NCS2005 (light capacitive load 1nF)\nOPA350EA/OP1177ARM (up to 1µF, MSOP-8 pkg)\nLM8261 (unlimited capacitive load, lower precision)"
- note removed: "IR=30÷40nA\n@3.3V"
- note removed: "To drive light capacitive load use OPA388, NCS2005,\nOPA350EA/OPA2350EA (up to 1µF, MSOP-8 pkg)\nLM8261 (unlimited capacitive load, lower precision)"
- note removed: "any low-offset (<0.1mV),\nhigh output current OpAmp\n*high CLoad drive*\nOPA388, NCS2005 (light capacitive load)\nOPA350EA (up to 1µF, MSOP-8 pkg)\nLM8261 (unlimited capacitive load, lower precision)"
- moved on the sheet: C16, H1, H2, H3, H4, J11, J9, R28, R29, U6
