File: Hardware/APPMC-WSP80.sch (KiCad schematic (older format))
At the start: 83 parts, among them J1 + 30V max, J10 STLINK-V3, J101 ADC_C, J102 ADC_D, J14 VDD, J15 PWM, J16 ADC_B, J17 3.0V, J18 1.5V, J2 VOut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

Commit message: 2022-09
Other:
- note added: "any low-offset (<0.1mV),\nhigh output current OpAmp\n*high CLoad drive*\nOPA388, NCS2005 (light capacitive load)\nOPA350EA/OP1177ARM (up to 1µF, MSOP-8 pkg)\nLM8261 (unlimited capacitive load, lower precision)"
- note removed: "any low-offset (<0.1mV),\nhigh output current OpAmp\n*high CLoad drive*\nOPA388, NCS2005 (light capacitive load)\nOPA350EA (up to 1µF, MSOP-8 pkg)\nLM8261 (unlimited capacitive load, lower precision)"
Changed lines of the file:
@@
 Text Label 6550 2700 0    50   ~ 0
 ADC_D
-Text Notes 1650 7450 0    39   Italic 0
+Text Notes 1950 6650 0    39   Italic 0
 any P-CH Mosfet with\nVgs(th)max<2V, low Rds(on)\n-PMV100EPAR\n-NXV90EPR\n-SI2343CDS-T1-GE3\n-SI2307CDS-T1-E3\n-CPH3351-TL-W
 Text Notes 3600 6850 0    50   Italic 0
@@
 Text Label 900  5950 0    50   ~ 0
 3.0V
-Text Notes 500  6950 0    50   Italic 0
-any low-offset (<0.1mV),\nhigh output current OpAmp\n*high CLoad drive*\nOPA388, NCS2005 (light capacitive load)\nOPA350EA (up to 1µF, MSOP-8 pkg)\nLM8261 (unlimited capacitive load, lower precision)
+Text Notes 500  7000 0    50   Italic 0
+any low-offset (<0.1mV),\nhigh output current OpAmp\n*high CLoad drive*\nOPA388, NCS2005 (light capacitive load)\nOPA350EA/OP1177ARM (up to 1µF, MSOP-8 pkg)\nLM8261 (unlimited capacitive load, lower precision)
 $Comp
 L Device:C_Small C101
